Commit message: Missing updates to previous commit

File: src/slam_project/urdf/udacity_bot.xacro (robot description, xacro)
@@ -118,5 +118,5 @@
       <dynamics damping="1.0" friction="1.0"/>
     </joint>
-  <link name='camera'>
+  <link name='camera_rgbd'>
     <inertial>
       <mass value="0.1"/>
@@ -143,5 +143,5 @@
   <joint type="fixed" name="camera_joint">
     <origin xyz="0.2 0 0" rpy="0 0 0"/>
-    <child link="camera"/>
+    <child link="camera_rgbd"/>
     <parent link="chassis"/>
   </joint>
